Commit message: Bringup finished waiting for description PR

File: src/agl_description/urdf/andresito.urdf (robot description, URDF)
Before this commit: robot andresito, 7 links, 6 joints
Joints:
- joint base_joint: origin xyz=0.0 0.0 0 rpy=0 0 0 -> xyz=0 -0.21 0.0
- joint base_link_left_back_wheel: axis 0 0 1 -> 0 1 0; limit lower=-3.14159265359 upper=3.14159265359 effort=1000.0 velocity=0.01 -> (none); type fixed -> continuous
- joint base_link_left_front_wheel: axis 0 0 1 -> 0 1 0; limit lower=-3.14159265359 upper=3.14159265359 effort=1000.0 velocity=0.01 -> (none); type fixed -> continuous
- joint base_link_right_back_wheel: axis 0 0 1 -> 0 1 0; limit lower=-3.14159265359 upper=3.14159265359 effort=1000.0 velocity=0.01 -> (none); type fixed -> continuous
- joint base_link_right_front_wheel: axis 0 0 1 -> 0 1 0; limit lower=-3.14159265359 upper=3.14159265359 effort=1000.0 velocity=0.01 -> (none); type fixed -> continuous

File: src/agl_description/urdf/andresito.xacro (robot description, xacro)
@@ -40,35 +40,31 @@
   <!-- JOINTS -->
   <joint name="base_joint" type="fixed">
-    <origin xyz="0.0 0.0 0" rpy="0 0 0"/>
+    <origin xyz="0 -${robot_depth/2} ${wheels_height}"/>
     <parent link="base_footprint"/>
     <child link="base_link" />
   </joint>
-  <joint name="base_link_left_front_wheel" type="fixed">
+  <joint name="base_link_left_front_wheel" type="continuous">
     <parent link="base_link"/>
     <child link="left_front_wheel"/>
     <origin xyz="${robot_width/2} ${robot_depth/2} ${wheels_height}"/>
-    <axis xyz="0 0 1"/>
-    <limit lower="-3.14159265359" upper="3.14159265359" effort="1000.0" velocity="0.01" />
+    <axis xyz="0 1 0"/>
   </joint>
-  <joint name="base_link_left_back_wheel" type="fixed">
+  <joint name="base_link_left_back_wheel" type="continuous">
     <parent link="base_link"/>
     <child link="left_back_wheel"/>
     <origin xyz="${robot_width/2} -${robot_depth/2} ${wheels_height}"/>
-    <axis xyz="0 0 1"/>
-    <limit lower="-3.14159265359" upper="3.14159265359" effort="1000.0" velocity="0.01" />
+    <axis xyz="0 1 0"/>
   </joint>
-  <joint name="base_link_right_front_wheel" type="fixed">
+  <joint name="base_link_right_front_wheel" type="continuous">
     <parent link="base_link"/>
     <child link="right_front_wheel"/>
     <origin xyz="-${robot_width/2} ${robot_depth/2} ${wheels_height}"/>
-    <axis xyz="0 0 1"/>
-    <limit lower="-3.14159265359" upper="3.14159265359" effort="1000.0" velocity="0.01" />
+    <axis xyz="0 1 0"/>
   </joint>
-  <joint name="base_link_right_back_wheel" type="fixed">
+  <joint name="base_link_right_back_wheel" type="continuous">
     <parent link="base_link"/>
     <child link="right_back_wheel"/>
     <origin xyz="-${robot_width/2} -${robot_depth/2} ${wheels_height}"/>
-    <axis xyz="0 0 1"/>
-    <limit lower="-3.14159265359" upper="3.14159265359" effort="1000.0" velocity="0.01" />
+    <axis xyz="0 1 0"/>
   </joint>
   <joint name="base_link_laser" type="fixed">
@@ -77,5 +73,4 @@
     <origin xyz="0 0 ${robot_height}"/>
     <axis xyz="0 0 1"/>
-    <!-- <limit lower="-3.14159265359" upper="3.14159265359" effort="1000.0" velocity="0.01" /> -->
   </joint>
 </robot>

Commit message: imu_link addition

File: src/agl_description/urdf/andresito.urdf (robot description, URDF)
Before this commit: robot andresito, 7 links, 6 joints
Links:
- added link imu_link, mass 0.005; collision box size=0.0 0.0 0.0; visual box size=0.0 0.0 0.0
Joints:
- added joint imu_joint: type fixed, parent base_link, child imu_link, origin xyz=-0.646 0.0 -0.055 rpy=3.1415922 0 3.1415922

Commit message: Last changes with witimu (imu does not work properly)

File: src/agl_description/urdf/andresito.urdf (robot description, URDF)
Before this commit: robot andresito, 8 links, 7 joints
Joints:
- joint imu_joint: axis (none) -> 0 0 1; origin xyz=-0.646 0.0 -0.055 rpy=3.1415922 0 3.1415922 -> xyz=0.03 0 0.08

Commit message: Camera integrated, rqt tf correct, node correct

File: src/agl_description/urdf/andresito.urdf (robot description, URDF)
Before this commit: robot andresito, 8 links, 7 joints
Links:
- removed link imu_link
- added link camera_accel_frame
- added link camera_accel_optical_frame
- added link camera_bottom_screw_frame
- added link camera_color_frame
- added link camera_color_optical_frame
- added link camera_depth_frame
- added link camera_depth_optical_frame
- added link camera_gyro_frame
- added link camera_gyro_optical_frame
- added link camera_imu_optical_frame
- added link camera_infra1_frame
- added link camera_infra1_optical_frame
- added link camera_infra2_frame
- added link camera_infra2_optical_frame
- added link camera_link, mass 0.072; collision box size=0.026 0.124 0.029; visual mesh filename=file:///opt/ros/humble/share/realsense2_description/meshes/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 scale=0.001 0.001 0.001
- added link realsense_link
Joints:
- removed joint imu_joint
- added joint base_link_to_realsense_link: type fixed, parent base_link, child realsense_link, origin xyz=0.04 0.04 0.0 rpy=0 0 3.1415922, axis 0 1 1
- added joint camera_accel_joint: type fixed, parent camera_link, child camera_accel_frame, origin xyz=-0.01602 -0.03022 0.0074 rpy=0 0 0
- added joint camera_accel_optical_joint: type fixed, parent camera_accel_frame, child camera_accel_optical_frame, origin xyz=0 0 0 rpy=-1.5707963267948966 0 -1.5707963267948966
- added joint camera_color_joint: type fixed, parent camera_link, child camera_color_frame, origin xyz=0 -0.059 0 rpy=0 0 0
- added joint camera_color_optical_joint: type fixed, parent camera_color_frame, child camera_color_optical_frame, origin xyz=0 0 0 rpy=-1.5707963267948966 0 -1.5707963267948966
- added joint camera_depth_joint: type fixed, parent camera_link, child camera_depth_frame, origin xyz=0 0 0 rpy=0 0 0
- added joint camera_depth_optical_joint: type fixed, parent camera_depth_frame, child camera_depth_optical_frame, origin xyz=0 0 0 rpy=-1.5707963267948966 0 -1.5707963267948966
- added joint camera_gyro_joint: type fixed, parent camera_link, child camera_gyro_frame, origin xyz=-0.01602 -0.03022 0.0074 rpy=0 0 0
- added joint camera_gyro_optical_joint: type fixed, parent camera_gyro_frame, child camera_gyro_optical_frame, origin xyz=0 0 0 rpy=-1.5707963267948966 0 -1.5707963267948966
- added joint camera_imu_optical_joint: type fixed, parent camera_gyro_optical_frame, child camera_imu_optical_frame, origin xyz=0 0 0 rpy=0 0 0
- added joint camera_infra1_joint: type fixed, parent camera_link, child camera_infra1_frame, origin xyz=0 0.0 0 rpy=0 0 0
- added joint camera_infra1_optical_joint: type fixed, parent camera_infra1_frame, child camera_infra1_optical_frame, origin xyz=0 0 0 rpy=-1.5707963267948966 0 -1.5707963267948966
- added joint camera_infra2_joint: type fixed, parent camera_link, child camera_infra2_frame, origin xyz=0 -0.095 0 rpy=0 0 0
- added joint camera_infra2_optical_joint: type fixed, parent camera_infra2_frame, child camera_infra2_optical_frame, origin xyz=0 0 0 rpy=-1.5707963267948966 0 -1.5707963267948966
- added joint camera_joint: type fixed, parent realsense_link, child camera_bottom_screw_frame, origin xyz=0 0 0 rpy=0 0 0
- added joint camera_link_joint: type fixed, parent camera_bottom_screw_frame, child camera_link, origin xyz=0.011150000000000002 0.0475 0.0145 rpy=0 0 0

File: src/agl_description/urdf/andresito.xacro (robot description, xacro)
@@ -4,4 +4,5 @@
   <!-- PROPERTIES -->
   <xacro:include filename="properties.xacro" />
+  <xacro:property name="deg_to_rad"  value="0.01745329"/>
   <!-- MACROS -->
   <xacro:include filename="wheel.xacro" />
@@ -38,5 +39,10 @@
   <xacro:wheel side="right" position="front"/>
   <xacro:wheel side="right" position="back"/>
+  <!-- <odometry_frame>odom</odometry_frame> -->
   <!-- JOINTS -->
+  <!-- <joint name="odom_base_footprint" type="fixed">
+    <parent link="odom"/>
+    <child link="base_footprint" />
+  </joint> -->
   <joint name="base_joint" type="fixed">
     <origin xyz="0 -${robot_depth/2} ${wheels_height}"/>
@@ -74,3 +80,15 @@
     <axis xyz="0 0 1"/>
   </joint>
+  <!-- CAMERA LINKS and JOINT -->
+  <xacro:include filename="$(find realsense2_description)/urdf/_d455.urdf.xacro" />
+  <link name="${camera_link}" />
+  <xacro:sensor_d455 parent="${camera_link}" use_nominal_extrinsics="true">
+    <origin xyz="0 0 0" rpy="0 0 0"/>
+  </xacro:sensor_d455>
+  <joint name="base_link_to_${camera_link}" type="fixed">
+    <axis xyz="0 1 1"/>
+    <parent link="base_link"/>
+    <child link="${camera_link}"/>
+    <origin xyz="${camera_x} ${camera_y} ${camera_z}" rpy="0 0 ${camera_rotation_z}"/>
+  </joint>
 </robot>

File: src/agl_description/urdf/properties.xacro (robot description, xacro)
@@ -12,10 +12,11 @@
     <xacro:property name="wheel_radius" value="0.05" />
     <!-- CAMERA -->
-    <!-- <xacro:property name="camera_link" value="realsense_link" />
+    <xacro:property name="camera_size" value="0.01" />
+    <xacro:property name="camera_link" value="realsense_link" />
     <xacro:property name="camera_relative_to" value="puller_base" />
-    <xacro:property name="camera_x" value="-${puller_depth/2-0.03}" />
-    <xacro:property name="camera_y" value="0.0" />
-    <xacro:property name="camera_z" value="0.24" />
-    <xacro:property name="camera_rotation_z" value="${180*deg_to_rad}" /> -->
+    <xacro:property name="camera_x" value="0.04" />
+    <xacro:property name="camera_y" value="0.04" />
+    <xacro:property name="camera_z" value="0.0" />
+    <xacro:property name="camera_rotation_z" value="${180*deg_to_rad}" />
     <!-- PROPERTIES -->
     <material name="blue">

Commit message: Few changes for slam

File: src/agl_description/urdf/andresito.urdf (robot description, URDF)
Before this commit: robot andresito, 23 links, 22 joints
Joints:
- removed joint base_joint
- added joint base_footprint_joint: type fixed, parent base_link, child base_footprint, origin xyz=0 0 0 rpy=0 0 0
- joint base_link_laser: origin xyz=0 0 0.08 -> xyz=0 0 0.08 rpy=0 0 3.1415922
- joint base_link_to_realsense_link: axis 0 1 1 -> 0 0 1; origin xyz=0.04 0.04 0.0 rpy=0 0 3.1415922 -> xyz=0.04 0.04 0.0

File: src/agl_description/urdf/andresito.xacro (robot description, xacro)
@@ -45,8 +45,13 @@
     <child link="base_footprint" />
   </joint> -->
-  <joint name="base_joint" type="fixed">
+  <!-- <joint name="base_joint" type="fixed">
     <origin xyz="0 -${robot_depth/2} ${wheels_height}"/>
     <parent link="base_footprint"/>
     <child link="base_link" />
+  </joint> -->
+  <joint name="base_footprint_joint" type="fixed">
+    <parent link="base_link"/>
+    <child link="base_footprint"/>
+    <origin xyz="0 0 0" rpy="0 0 0"/>
   </joint>
   <joint name="base_link_left_front_wheel" type="continuous">
@@ -77,5 +82,5 @@
     <parent link="base_link"/>
     <child link="laser"/>
-    <origin xyz="0 0 ${robot_height}"/>
+    <origin xyz="0 0 ${robot_height}" rpy="0 0 ${camera_rotation_z}"/>
     <axis xyz="0 0 1"/>
   </joint>
@@ -87,8 +92,9 @@
   </xacro:sensor_d455>
   <joint name="base_link_to_${camera_link}" type="fixed">
-    <axis xyz="0 1 1"/>
+    <axis xyz="0 0 1"/>
     <parent link="base_link"/>
     <child link="${camera_link}"/>
-    <origin xyz="${camera_x} ${camera_y} ${camera_z}" rpy="0 0 ${camera_rotation_z}"/>
+    <!-- <origin xyz="${camera_x} ${camera_y} ${camera_z}" rpy="0 0 ${camera_rotation_z}"/> -->
+    <origin xyz="${camera_x} ${camera_y} ${camera_z}"/>
   </joint>
 </robot>
